File: kicad/plant_station/plant_station_v3.kicad_pcb (KiCad board)
At the start: 2 copper layers, 160.8 x 185 mm, 95 parts, among them IC1 VEML7700-TT, IC3 TLC555CDR, IC4 ADC081C021CIMK_NOPB, J1 Conn_02x08_Odd_Even, J10 I2C HOST, J11 SOIL_I2C, J12 WEATHER_I2C, J13 MB_I2C, J14 Ambient_Led_6, J15 Ambient_Led_5, J16 Conn_01x06, J17 GPIO, J18 ALWAYS_ON, J19 Ammeter_Jumper, J2 MB_I2C, J20 LED_I2C, J4 MB_I2C, J5 MB_I2C, J6 MB_I2C, J7 Conn_01x08, J8 UART, J9 I2C SCREEN, P1 USB_C_Plug_USB2.0, Q1 DTC113Z, Q3 DTC113Z, Q4 DMG2301L, Q5 BC817DS,115, U1 HDC2010YPAT, U4 ESP-WROOM-02, U5 TPL5110, U6 CP2102N-A01-GQFN28

Commit message: pcb v3 sent to production and the first attempts to design the enclosure
Parts:
- removed the REF** at (220.9, 46.5)
- removed the REF** at (207.2, 62.7)
- removed the REF** at (186.0, 61.0)
- removed the REF** at (185.9, 43.4)
- removed the REF** at (185.9, 25.9)
- added REF**: Drill Hole, Parts:Drill Hole, F.Cu at (112.4, 89.0)
- added REF**: Drill Hole, Parts:Drill Hole, F.Cu at (118.7, 91.0)
- added REF**: Drill Hole, Parts:Drill Hole, F.Cu at (118.7, 90.0)
- added REF**: Drill Hole, Parts:Drill Hole, F.Cu at (118.7, 89.0)
- added REF**: Drill Hole, Parts:Drill Hole, F.Cu at (152.0, 80.3)
- added REF**: Drill Hole, Parts:Drill Hole, F.Cu at (153.0, 80.3)
- added REF**: Drill Hole, Parts:Drill Hole, F.Cu at (154.0, 80.3)
- added REF**: Drill Hole, Parts:Drill Hole, F.Cu at (155.0, 80.3)
- added REF**: Drill Hole, Parts:Drill Hole, F.Cu at (156.0, 80.3)
- added REF**: Drill Hole, Parts:Drill Hole, F.Cu at (157.0, 80.3)
- added REF**: Drill Hole, Parts:Drill Hole, F.Cu at (157.0, 84.7)
- added REF**: Drill Hole, Parts:Drill Hole, F.Cu at (112.5, 90.0)
- added REF**: Drill Hole, Parts:Drill Hole, F.Cu at (156.0, 84.7)
- added REF**: Drill Hole, Parts:Drill Hole, F.Cu at (155.0, 84.7)
- added REF**: Drill Hole, Parts:Drill Hole, F.Cu at (154.0, 84.7)
- added REF**: Drill Hole, Parts:Drill Hole, F.Cu at (153.0, 84.7)
- added REF**: Drill Hole, Parts:Drill Hole, F.Cu at (152.0, 84.7)
- added REF**: Drill Hole, Parts:Drill Hole, F.Cu at (180.2, 79.9)
- added REF**: Drill Hole, Parts:Drill Hole, F.Cu at (181.1, 80.2)
- added REF**: Drill Hole, Parts:Drill Hole, F.Cu at (182.1, 80.3)
- added REF**: Drill Hole, Parts:Drill Hole, F.Cu at (183.1, 80.3)
- added REF**: Drill Hole, Parts:Drill Hole, F.Cu at (184.1, 80.2)
- added REF**: Drill Hole, Parts:Drill Hole, F.Cu at (112.6, 91.0)
- added REF**: Drill Hole, Parts:Drill Hole, F.Cu at (185.0, 79.9)
- added REF**: Drill Hole, Parts:Drill Hole, F.Cu at (185.0, 84.7)
- added REF**: Drill Hole, Parts:Drill Hole, F.Cu at (184.0, 84.7)
- added REF**: Drill Hole, Parts:Drill Hole, F.Cu at (183.0, 84.7)
- added REF**: Drill Hole, Parts:Drill Hole, F.Cu at (182.0, 84.7)
- added REF**: Drill Hole, Parts:Drill Hole, F.Cu at (181.0, 84.7)
- added REF**: Drill Hole, Parts:Drill Hole, F.Cu at (180.0, 84.7)
- added REF**: Drill Hole, Parts:Drill Hole, F.Cu at (216.0, 80.3)
- added REF**: Drill Hole, Parts:Drill Hole, F.Cu at (215.0, 80.3)
- added REF**: Drill Hole, Parts:Drill Hole, F.Cu at (214.0, 80.3)
- added REF**: Drill Hole, Parts:Drill Hole, F.Cu at (112.6, 92.0)
- added REF**: Drill Hole, Parts:Drill Hole, F.Cu at (213.0, 80.3)
- added REF**: Drill Hole, Parts:Drill Hole, F.Cu at (212.0, 80.3)
- added REF**: Drill Hole, Parts:Drill Hole, F.Cu at (211.0, 80.3)
- added REF**: Drill Hole, Parts:Drill Hole, F.Cu at (216.0, 84.7)
- added REF**: Drill Hole, Parts:Drill Hole, F.Cu at (215.0, 84.7)
- added REF**: Drill Hole, Parts:Drill Hole, F.Cu at (214.0, 84.7)
- added REF**: Drill Hole, Parts:Drill Hole, F.Cu at (213.0, 84.7)
- added REF**: Drill Hole, Parts:Drill Hole, F.Cu at (212.0, 84.7)
- added REF**: Drill Hole, Parts:Drill Hole, F.Cu at (211.0, 84.7)
- added REF**: MountingHole_2.2mm_M2_ISO7380, MountingHole:MountingHole_2.2mm_M2_ISO7380, F.Cu at (167.0, 61.0)
- added REF**: Drill Hole, Parts:Drill Hole, F.Cu at (112.5, 93.0)
- added REF**: MountingHole_2.2mm_M2_ISO7380, MountingHole:MountingHole_2.2mm_M2_ISO7380, F.Cu at (121.5, 73.2)
- added REF**: MountingHole_2.2mm_M2_ISO7380, MountingHole:MountingHole_2.2mm_M2_ISO7380, F.Cu at (131.2, 92.0)
- added REF**: MountingHole_2.2mm_M2_ISO7380, MountingHole:MountingHole_2.2mm_M2_ISO7380, F.Cu at (121.5, 111.0)
- added REF**: MountingHole_2.2mm_M2_ISO7380, MountingHole:MountingHole_2.2mm_M2_ISO7380, F.Cu at (107.3, 98.8)
- added REF**: MountingHole_2.2mm_M2_ISO7380, MountingHole:MountingHole_2.2mm_M2_ISO7380, F.Cu at (88.5, 108.5)
- added REF**: MountingHole_2.2mm_M2_ISO7380, MountingHole:MountingHole_2.2mm_M2_ISO7380, F.Cu at (69.6, 98.8)
- added REF**: MountingHole_2.2mm_M2_ISO7380, MountingHole:MountingHole_2.2mm_M2_ISO7380, F.Cu at (76.2, 82.6)
- added REF**: MountingHole_2.2mm_M2_ISO7380, MountingHole:MountingHole_2.2mm_M2_ISO7380, F.Cu at (82.9, 66.5)
- added REF**: Drill Hole, Parts:Drill Hole, F.Cu at (112.4, 94.0)
- added REF**: Drill Hole, Parts:Drill Hole, F.Cu at (118.7, 94.0)
- added REF**: Drill Hole, Parts:Drill Hole, F.Cu at (118.7, 93.0)
- added REF**: Drill Hole, Parts:Drill Hole, F.Cu at (118.7, 92.0)
- moved IC1 182.2 mm to (176.5, 73.8), turned to 0 degrees
- moved C14 179.0 mm to (180.0, 76.6), turned to 0 degrees
- moved C13 171.0 mm to (184.8, 76.6), turned to 180 degrees
- moved J12 170.1 mm to (182.5, 72.2), turned to 0 degrees
- moved Q3 166.6 mm to (182.5, 68.6), turned to 270 degrees
- moved U1 164.6 mm to (186.0, 72.6), turned to 90 degrees
- moved FB1 159.9 mm to (123.4, 88.5), turned to 180 degrees
- moved Ra1 157.7 mm to (124.0, 77.7), turned to 180 degrees
- moved Rb1 155.7 mm to (124.0, 80.2), turned to 0 degrees
- moved C3 155.7 mm to (123.4, 82.7), turned to 0 degrees
- moved C7 154.0 mm to (123.4, 85.3), turned to 180 degrees
- moved D10 153.4 mm to (123.5, 91.8), turned to 0 degrees
- moved Cref1 152.0 mm to (129.0, 77.7), turned to 0 degrees
- moved Q1 152.0 mm to (123.4, 94.5), turned to 0 degrees
- moved J11 151.2 mm to (125.2, 92.1), turned to 270 degrees
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Connections:
- J14 pad 1: /leds/LED_6_B -> /leds/LED_3_B
- J14 pad 2: /leds/LED_6_G -> /leds/LED_3_G
- J14 pad 3: /leds/LED_6_R -> /leds/LED_3_R
- J14 pad 6: Net-(J14-Pad5) -> Net-(J14-Pad6)
- J15 pad 1: /leds/LED_1_B -> /leds/LED_4_B
- J15 pad 2: /leds/LED_1_G -> /leds/LED_4_G
- J15 pad 3: /leds/LED_1_R -> /leds/LED_4_R
- J15 pad 5: Net-(J14-Pad5) -> Net-(J15-Pad5)
- J15 pad 6: Net-(J14-Pad5) -> Net-(J15-Pad6)
- J20 pad MP1: Net-(J14-Pad5) -> Net-(J20-PadMP1)
- J20 pad MP2: Net-(J14-Pad5) -> Net-(J20-PadMP2)
- LED1 pad C1: /leds/LED_2_B -> /leds/LED_1_B
- LED1 pad C2: /leds/LED_2_G -> /leds/LED_1_G
- LED1 pad C3: /leds/LED_2_R -> /leds/LED_1_R
- LED2 pad C1: /leds/LED_3_B -> /leds/LED_2_B
- LED2 pad C2: /leds/LED_3_G -> /leds/LED_2_G
- LED2 pad C3: /leds/LED_3_R -> /leds/LED_2_R
- LED3 pad C1: /leds/LED_4_B -> /leds/LED_5_B
- LED3 pad C2: /leds/LED_4_G -> /leds/LED_5_G
- LED3 pad C3: /leds/LED_4_R -> /leds/LED_5_R
- LED4 pad C1: /leds/LED_5_B -> /leds/LED_6_B
- LED4 pad C2: /leds/LED_5_G -> /leds/LED_6_G
- LED4 pad C3: /leds/LED_5_R -> /leds/LED_6_R
- P1 pad B6: (no net) -> /usb_serial/D+
- P1 pad B7: (no net) -> /usb_serial/D-
Routing:
- net Net-(J14-Pad5): track 39.1 -> 0.00 mm
- net VDD: track 243.9 -> 266.7 mm
- net Net-(P1-PadS1): track 0.00 -> 19.5 mm
- net /moisture_sensor/VA: track 5.42 -> 20.2 mm, vias 5 -> 2
- net /leds/LED_3_B: track 24.7 -> 10.4 mm, vias 1 -> 0
- net /leds/SDA: track 6.59 -> 20.4 mm, vias 2 -> 0
- net /leds/LED_3_G: track 21.8 -> 9.83 mm, vias 1 -> 0
- net /leds/LED_4_R: track 20.0 -> 8.63 mm, vias 1 -> 0
- net /leds/SCL: track 6.10 -> 17.4 mm, vias 2 -> 0
- net /leds/LED_4_B: track 16.3 -> 5.23 mm, vias 1 -> 0
- net /leds/LED_4_G: track 18.1 -> 7.21 mm, vias 1 -> 0
- net /leds/LED_1_R: track 11.5 -> 2.73 mm, vias 0 -> 1
- net GND: track 320.4 -> 312.1 mm, vias 24 -> 23
- net /leds/LED_1_G: track 10.6 -> 3.86 mm, vias 0 -> 1
- net /moisture_sensor/GNDA: track 26.1 -> 19.5 mm, vias 4 -> 11
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- added copper zone on B.Cu, net /moisture_sensor/GNDA
- added copper zone on B.Cu, net /moisture_sensor/Sensor_Inside
- added copper zone on F.Cu, net /moisture_sensor/Sensor_Inside
- added copper zone on F.Cu, net /moisture_sensor/VA
- removed copper zone on F.Cu, net (none)
- removed copper zone on B.Cu, net /moisture_sensor/VA
Other:
- board size 160.8 x 185 mm -> 174.4 x 59.3 mm
- board text added: "The hole on the LEDs screen! :("

Commit message: Pre-refactoring, diagnostics complete, timer not working properly
Other:
- board text added: "The hole on the LEDs screen is missing. And mirror the holes!"
- board text removed: "The hole on the LEDs screen! :("
