File: kicad/plant_station.sch (KiCad schematic (older format))
At the start: 12 parts, among them J10 I2C HOST, J13 MB_I2C, J2 MB_I2C, J4 MB_I2C, J5 MB_I2C, J6 MB_I2C, J9 I2C SCREEN

Commit message: Libraries cleanup
Other:
- note removed: "VDD - Always powered 3v3\n3v3 - Timer-backed power source, this should be used to make sure the component is not powered when the device is sleeping\nVA - Only used in Soil Moisture Sensor for power filtered by Ferrite Beads"
- moved on the sheet: J10, J9
Changed lines of the file:
@@
 $Descr A4 11693 8268
 encoding utf-8
-Sheet 1 6
+Sheet 1 7
 Title ""
 Date ""
@@
 Comment4 ""
 $EndDescr
-$Comp
-L power:PWR_FLAG #FLG0101
-U 1 1 611E169D
-P 10550 800
-F 0 "#FLG0101" H 10550 875 50  0001 C CNN
-F 1 "PWR_FLAG" H 10550 973 50  0000 C CNN
-F 2 "" H 10550 800 50  0001 C CNN
-F 3 "~" H 10550 800 50  0001 C CNN
-	1    10550 800
-	1    0    0    -1
-$EndComp
-$Comp
-L power:PWR_FLAG #FLG0102
-U 1 1 611E1B09
-P 10950 800
-F 0 "#FLG0102" H 10950 875 50  0001 C CNN
-F 1 "PWR_FLAG" H 10950 973 50  0000 C CNN
-F 2 "" H 10950 800 50  0001 C CNN
-F 3 "~" H 10950 800 50  0001 C CNN
-	1    10950 800
-	1    0    0    -1
-$EndComp
-$Comp
-L power:GND #PWR0134
-U 1 1 611E3051
-P 10950 800
-F 0 "#PWR0134" H 10950 550 50  0001 C CNN
-F 1 "GND" H 10955 627 50  0000 C CNN
-F 2 "" H 10950 800 50  0001 C CNN
-F 3 "" H 10950 800 50  0001 C CNN
-	1    10950 800
-	1    0    0    -1
-$EndComp
-$Comp
-L power:+3V3 #PWR0133
-U 1 1 611E24F6
-P 10550 800
-F 0 "#PWR0133" H 10550 650 50  0001 C CNN
-F 1 "+3V3" H 10565 973 50  0000 C CNN
-F 2 "" H 10550 800 50  0001 C CNN
-F 3 "" H 10550 800 50  0001 C CNN
-	1    10550 800
-	-1   0    0    1
-$EndComp
 Text Notes 2200 1650 0    50   ~ 0
 usb breakout\n+tantalum decouplers\n+fix the probe\nleds board + ambient leds\nsensor board\noscillator???\n-look for a different humidity sensor\nstack boards\n+power schematics\n+analog VCC on ADC\n+sleep/wake bus
@@
 F5 "HOST_WAKE_UP" I L 7700 2350 50
 $EndSheet
-Text Label 850  7050 1    50   ~ 0
-SDA
-Text Label 950  7050 1    50   ~ 0
+Text Label 1200 5850 1    50   ~ 0
+SDA
+Text Label 1300 5850 1    50   ~ 0
 SCL
 $Comp
 L power:GND #PWR0140
 U 1 1 5FCFC642
-P 1150 7050
-F 0 "#PWR0140" H 1150 6800 50  0001 C CNN
-F 1 "GND" V 1150 6850 50  0000 C CNN
-F 2 "" H 1150 7050 50  0001 C CNN
-F 3 "" H 1150 7050 50  0001 C CNN
-	1    1150 7050
+P 1500 5850
+F 0 "#PWR0140" H 1500 5600 50  0001 C CNN
+F 1 "GND" V 1500 5650 50  0000 C CNN
+F 2 "" H 1500 5850 50  0001 C CNN
+F 3 "" H 1500 5850 50  0001 C CNN
+	1    1500 5850
 	-1   0    0    1
 $EndComp
@@
 Text Label 8600 2250 0    50   ~ 0
 SDA
-Text Label 1400 7050 1    50   ~ 0
-SDA
-Text Label 1500 7050 1    50   ~ 0
+Text Label 1750 5850 1    50   ~ 0
+SDA
+Text Label 1850 5850 1    50   ~ 0
 SCL
 $Comp
 L power:GND #PWR0138
 U 1 1 5FB01C12
-P 1700 7050
-F 0 "#PWR0138" H 1700 6800 50  0001 C CNN
-F 1 "GND" V 1700 6850 50  0000 C CNN
-F 2 "" H 1700 7050 50  0001 C CNN
-F 3 "" H 1700 7050 50  0001 C CNN
-	1    1700 7050
+P 2050 5850
+F 0 "#PWR0138" H 2050 5600 50  0001 C CNN
+F 1 "GND" V 2050 5650 50  0000 C CNN
+F 2 "" H 2050 5850 50  0001 C CNN
+F 3 "" H 2050 5850 50  0001 C CNN
+	1    2050 5850
 	-1   0    0    1
 $EndComp
@@
 L Connector_Generic:Conn_01x04 J10
 U 1 1 5FAF3653
-P 1600 7250
-F 0 "J10" V 1600 6850 50  0000 L CNN
-F 1 "I2C HOST" V 1750 7000 50  0000 L CNN
-F 2 "Connector_PinSocket_2.54mm:PinSocket_1x04_P2.54mm_Vertical" H 1600 7250 50  0001 C CNN
-F 3 "~" H 1600 7250 50  0001 C CNN
-F 4 "Samtec SLW-104-01-T-S" V 1600 7250 50  0001 C CNN "Field4"
-	1    1600 7250
+P 1950 6050
+F 0 "J10" V 1950 5650 50  0000 L CNN
+F 1 "I2C HOST" V 2100 5800 50  0000 L CNN
+F 2 "Connector_PinSocket_2.54mm:PinSocket_1x04_P2.54mm_Vertical" H 1950 6050 50  0001 C CNN
+F 3 "~" H 1950 6050 50  0001 C CNN
+F 4 "Samtec SLW-104-01-T-S" V 1950 6050 50  0001 C CNN "Field4"
+	1    1950 6050
 	0    1    1    0
 $EndComp
@@
 L power:VDD #PWR012
 U 1 1 5FA09D29
-P 1600 7050
-F 0 "#PWR012" H 1600 6900 50  0001 C CNN
-F 1 "VDD" V 1600 7250 50  0000 C CNN
-F 2 "" H 1600 7050 50  0001 C CNN
-F 3 "" H 1600 7050 50  0001 C CNN
-	1    1600 7050
-	1    0    0    -1
-$EndComp
-$Comp
-L power:PWR_FLAG #FLG01
-U 1 1 5FAB0070
-P 10150 800
-F 0 "#FLG01" H 10150 875 50  0001 C CNN
-F 1 "PWR_FLAG" H 10150 973 50  0000 C CNN
-F 2 "" H 10150 800 50  0001 C CNN
-F 3 "~" H 10150 800 50  0001 C CNN
-	1    10150 800
-	1    0    0    -1
-$EndComp
-$Comp
-L power:VDD #PWR027
-U 1 1 5FAB03BE
-P 10150 800
-F 0 "#PWR027" H 10150 650 50  0001 C CNN
-F 1 "VDD" H 10165 973 50  0000 C CNN
-F 2 "" H 10150 800 50  0001 C CNN
-F 3 "" H 10150 800 50  0001 C CNN
-	1    10150 800
-	-1   0    0    1
+P 1950 5850
+F 0 "#PWR012" H 1950 5700 50  0001 C CNN
+F 1 "VDD" V 1950 6050 50  0000 C CNN
+F 2 "" H 1950 5850 50  0001 C CNN
+F 3 "" H 1950 5850 50  0001 C CNN
+	1    1950 5850
+	1    0    0    -1
 $EndComp
 $Comp
 L Connector_Generic:Conn_01x04 J9
 U 1 1 5FCFC63C
-P 1050 7250
-F 0 "J9" V 1050 6850 50  0000 L CNN
-F 1 "I2C SCREEN" V 1200 6950 50  0000 L CNN
-F 2 "Connector_PinSocket_2.54mm:PinSocket_1x04_P2.54mm_Vertical" H 1050 7250 50  0001 C CNN
-F 3 "~" H 1050 7250 50  0001 C CNN
-F 4 "Samtec SLW-104-01-T-S" V 1050 7250 50  0001 C CNN "Field4"
-	1    1050 7250
+P 1400 6050
+F 0 "J9" V 1400 5650 50  0000 L CNN
+F 1 "I2C SCREEN" V 1550 5750 50  0000 L CNN
+F 2 "Connector_PinSocket_2.54mm:PinSocket_1x04_P2.54mm_Vertical" H 1400 6050 50  0001 C CNN
+F 3 "~" H 1400 6050 50  0001 C CNN
+F 4 "Samtec SLW-104-01-T-S" V 1400 6050 50  0001 C CNN "Field4"
+	1    1400 6050
 	0    1    1    0
 $EndComp
@@
 L power:VDD #PWR02
 U 1 1 5FAB4B8A
-P 1050 7050
-F 0 "#PWR02" H 1050 6900 50  0001 C CNN
-F 1 "VDD" V 1050 7250 50  0000 C CNN
-F 2 "" H 1050 7050 50  0001 C CNN
-F 3 "" H 1050 7050 50  0001 C CNN
-	1    1050 7050
+P 1400 5850
+F 0 "#PWR02" H 1400 5700 50  0001 C CNN
+F 1 "VDD" V 1400 6050 50  0000 C CNN
+F 2 "" H 1400 5850 50  0001 C CNN
+F 3 "" H 1400 5850 50  0001 C CNN
+	1    1400 5850
 	1    0    0    -1
 $EndComp
@@
 NoConn ~ 2400 2450
 NoConn ~ 2400 2350
-Text Notes 4700 950  0    50   ~ 0
-VDD - Always powered 3v3\n3v3 - Timer-backed power source, this should be used to make sure the component is not powered when the device is sleeping\nVA - Only used in Soil Moisture Sensor for power filtered by Ferrite Beads
+$Sheet
+S 1550 6850 900  550
+U 610543CF
+F0 "charger" 50
+F1 "charger.sch" 50
+$EndSheet
 $EndSCHEMATC

Commit message: Schematics cleanup
Parts:
- removed D12, D13, D8, D9: LS4148, Parts:MELF_SOD_80_3_BZT55B13GS08, symbol Device:D_Small
- removed J10: I2C HOST, Connector_PinSocket_2.54mm:PinSocket_1x04_P2.54mm_Vertical, symbol Connector_Generic:Conn_01x04
- J9: value I2C SCREEN -> I2C
Connections:
- net ALL_EN: now also D6.1 (K), J13.6, J2.6, J4.6, J5.6, J6.6; no longer D6.2 (A)
- net HOST_WAKE renamed HOST_WAKE_UP
- net VDD renamed +3V3
- new net esp8266/ALL_EN: D6.2 (A)
Other:
- note added: "VCC - Power from Source\nGNDPWR - Ground from Source\n3v3 - Regulated 3.3v\nGND - Digital Ground"
- moved on the sheet: D6, J4, J9

Commit message: Comitting yesterday's leftovers
Parts:
- renumbered D6 to D1, J2 to J1, J5 to J2, J4 to J3, J6 to J4, J13 to J5, J9 to J6
Changed lines of the file:
@@
 F9 "BOOT_MODE" I L 7700 3050 50
 F10 "BATT_GAUGE_SHDN" O R 8600 3350 50
+F11 "nCH_PGOOD" I R 8600 3250 50
 $EndSheet
 Text Label 1850 4650 2    50   ~ 0
@@
 SCL
 $Comp
-L power:GND #PWR0140
+L power:GND #PWR012
 U 1 1 5FCFC642
 P 1850 4350
-F 0 "#PWR0140" H 1850 4100 50  0001 C CNN
+F 0 "#PWR012" H 1850 4100 50  0001 C CNN
 F 1 "GND" V 1850 4100 50  0000 C CNN
 F 2 "" H 1850 4350 50  0001 C CNN
@@
 $EndSheet
 $Comp
-L power:GND #PWR01
+L power:GND #PWR03
 U 1 1 6027ED70
 P 1500 2350
-F 0 "#PWR01" H 1500 2100 50  0001 C CNN
+F 0 "#PWR03" H 1500 2100 50  0001 C CNN
 F 1 "GND" V 1505 2222 50  0000 R CNN
 F 2 "" H 1500 2350 50  0001 C CNN
@@
 ALL_EN
 $Comp
-L Device:D_Small D6
+L Device:D_Small D1
 U 1 1 603E1FEA
 P 8750 2800
-F 0 "D6" H 8650 2750 50  0000 C CNN
+F 0 "D1" H 8650 2750 50  0000 C CNN
 F 1 "LS4148" H 8750 2916 50  0001 C CNN
 F 2 "Parts:MELF_SOD_80_3_BZT55B13GS08" V 8750 2800 50  0001 C CNN
@@
 HOST_WAKE_UP
 $Comp
-L power:GND #PWR09
+L power:GND #PWR04
 U 1 1 60493E6F
 P 3050 2350
-F 0 "#PWR09" H 3050 2100 50  0001 C CNN
+F 0 "#PWR04" H 3050 2100 50  0001 C CNN
 F 1 "GND" V 3055 2222 50  0000 R CNN
 F 2 "" H 3050 2350 50  0001 C CNN
@@
 HOST_WAKE_UP
 $Comp
-L power:GND #PWR011
+L power:GND #PWR08
 U 1 1 60496837
 P 3050 3300
-F 0 "#PWR011" H 3050 3050 50  0001 C CNN
+F 0 "#PWR08" H 3050 3050 50  0001 C CNN
 F 1 "GND" V 3055 3172 50  0000 R CNN
 F 2 "" H 3050 3300 50  0001 C CNN
@@
 $EndSheet
 $Comp
-L Connector_Generic:Conn_01x04 J9
+L Connector_Generic:Conn_01x04 J6
 U 1 1 5FCFC63C
 P 2050 4450
-F 0 "J9" H 1950 4650 50  0000 L CNN
+F 0 "J6" H 1950 4650 50  0000 L CNN
 F 1 "I2C" H 2050 4650 50  0000 L CNN
 F 2 "Connector_PinSocket_2.54mm:PinSocket_1x04_P2.54mm_Vertical" H 2050 4450 50  0001 C CNN
@@
 $EndComp
 $Comp
-L power:GND #PWR05
+L power:GND #PWR07
 U 1 1 5F3DEF4D
 P 1500 3300
-F 0 "#PWR05" H 1500 3050 50  0001 C CNN
+F 0 "#PWR07" H 1500 3050 50  0001 C CNN
 F 1 "GND" V 1505 3172 50  0000 R CNN
 F 2 "" H 1500 3300 50  0001 C CNN
@@
 HOST_WAKE_UP
 $Comp
-L Parts:505567-0671 J4
+L Parts:505567-0671 J3
 U 1 1 5F3DEF65
 P 1500 3300
-F 0 "J4" H 1750 3450 50  0000 C CNN
+F 0 "J3" H 1750 3450 50  0000 C CNN
 F 1 "MB_I2C" H 1950 3450 50  0000 C CNN
 F 2 "Parts:Molex_Conn_SMD_01x06_505567_0671" H 2250 3400 50  0001 L CNN
@@
 $EndComp
 $Comp
-L power:GND #PWR08
+L power:GND #PWR011
 U 1 1 5F3DEF6D
 P 3050 4250
-F 0 "#PWR08" H 3050 4000 50  0001 C CNN
+F 0 "#PWR011" H 3050 4000 50  0001 C CNN
 F 1 "GND" V 3055 4122 50  0000 R CNN
 F 2 "" H 3050 4250 50  0001 C CNN
@@
 HOST_WAKE_UP
 $Comp
-L Parts:505567-0671 J13
+L Parts:505567-0671 J5
 U 1 1 5F3DEF85
 P 3050 4250
-F 0 "J13" H 3350 4400 50  0000 C CNN
+F 0 "J5" H 3350 4400 50  0000 C CNN
 F 1 "MB_I2C" H 3550 4400 50  0000 C CNN
 F 2 "Parts:Molex_Conn_SMD_01x06_505567_0671" H 3800 4350 50  0001 L CNN
@@
 $EndComp
 $Comp
-L Parts:505567-0671 J2
+L Parts:505567-0671 J1
 U 1 1 6045DC89
 P 1500 2350
-F 0 "J2" H 1750 2500 50  0000 C CNN
+F 0 "J1" H 1750 2500 50  0000 C CNN
 F 1 "MB_I2C" H 1950 2500 50  0000 C CNN
 F 2 "Parts:Molex_Conn_SMD_01x06_505567_0671" H 2250 2450 50  0001 L CNN
@@
 $EndComp
 $Comp
-L Parts:505567-0671 J5
+L Parts:505567-0671 J2
 U 1 1 60493E8D
 P 3050 2350
-F 0 "J5" H 3300 2500 50  0000 C CNN
+F 0 "J2" H 3300 2500 50  0000 C CNN
 F 1 "MB_I2C" H 3500 2500 50  0000 C CNN
 F 2 "Parts:Molex_Conn_SMD_01x06_505567_0671" H 3800 2450 50  0001 L CNN
@@
 $EndComp
 $Comp
-L Parts:505567-0671 J6
+L Parts:505567-0671 J4
 U 1 1 60496855
 P 3050 3300
-F 0 "J6" H 3300 3450 50  0000 C CNN
+F 0 "J4" H 3300 3450 50  0000 C CNN
 F 1 "MB_I2C" H 3500 3450 50  0000 C CNN
 F 2 "Parts:Molex_Conn_SMD_01x06_505567_0671" H 3800 3400 50  0001 L CNN
@@
 F6 "USB_CHR1" I R 6250 2950 50
 F7 "SDA" B L 5350 2850 50
+F8 "nCH_PGOOD" O L 5350 3050 50
 $EndSheet
 Text Notes 9550 1650 0    50   ~ 0
@@
 P 9900 950
 AR Path="/5F48275C/617B518B" Ref="#PWR?"  Part="1"
-AR Path="/617B518B" Ref="#PWR?"  Part="1"
-F 0 "#PWR?" H 9900 700 50  0001 C CNN
+AR Path="/617B518B" Ref="#PWR01"  Part="1"
+F 0 "#PWR01" H 9900 700 50  0001 C CNN
 F 1 "GND" H 9905 777 50  0000 C CNN
 F 2 "" H 9900 950 50  0001 C CNN
@@
 P 10250 950
 AR Path="/5F48275C/617B5197" Ref="#PWR?"  Part="1"
-AR Path="/617B5197" Ref="#PWR?"  Part="1"
-F 0 "#PWR?" H 10250 750 50  0001 C CNN
+AR Path="/617B5197" Ref="#PWR02"  Part="1"
+F 0 "#PWR02" H 10250 750 50  0001 C CNN
 F 1 "GNDPWR" H 10254 796 50  0000 C CNN
 F 2 "" H 10250 900 50  0001 C CNN
@@
 	5200 3150 5350 3150
 $Comp
-L power:+3V3 #PWR?
+L power:+3V3 #PWR05
 U 1 1 619A414D
 P 1500 2450
-F 0 "#PWR?" H 1500 2300 50  0001 C CNN
+F 0 "#PWR05" H 1500 2300 50  0001 C CNN
 F 1 "+3V3" V 1515 2578 50  0000 L CNN
 F 2 "" H 1500 2450 50  0001 C CNN
@@
 $EndComp
 $Comp
-L power:+3V3 #PWR?
+L power:+3V3 #PWR06
 U 1 1 619A4748
 P 3050 2450
-F 0 "#PWR?" H 3050 2300 50  0001 C CNN
+F 0 "#PWR06" H 3050 2300 50  0001 C CNN
 F 1 "+3V3" V 3065 2578 50  0000 L CNN
 F 2 "" H 3050 2450 50  0001 C CNN
@@
 $EndComp
 $Comp
-L power:+3V3 #PWR?
+L power:+3V3 #PWR010
 U 1 1 619A4B96
 P 3050 3400
-F 0 "#PWR?" H 3050 3250 50  0001 C CNN
+F 0 "#PWR010" H 3050 3250 50  0001 C CNN
 F 1 "+3V3" V 3065 3528 50  0000 L CNN
 F 2 "" H 3050 3400 50  0001 C CNN
@@
 $EndComp
 $Comp
-L power:+3V3 #PWR?
+L power:+3V3 #PWR013
 U 1 1 619A4F33
 P 3050 4350
-F 0 "#PWR?" H 3050 4200 50  0001 C CNN
+F 0 "#PWR013" H 3050 4200 50  0001 C CNN
 F 1 "+3V3" V 3065 4478 50  0000 L CNN
 F 2 "" H 3050 4350 50  0001 C CNN
@@
 $EndComp
 $Comp
-L power:+3V3 #PWR?
+L power:+3V3 #PWR09
 U 1 1 619A517D
 P 1500 3400
-F 0 "#PWR?" H 1500 3250 50  0001 C CNN
+F 0 "#PWR09" H 1500 3250 50  0001 C CNN
 F 1 "+3V3" V 1515 3528 50  0000 L CNN
 F 2 "" H 1500 3400 50  0001 C CNN
@@
 $EndComp
 $Comp
-L power:+3V3 #PWR?
+L power:+3V3 #PWR014
 U 1 1 619AA26A
 P 1850 4450
-F 0 "#PWR?" H 1850 4300 50  0001 C CNN
+F 0 "#PWR014" H 1850 4300 50  0001 C CNN
 F 1 "+3V3" V 1850 4700 50  0000 C CNN
 F 2 "" H 1850 4450 50  0001 C CNN
@@
 	0    -1   -1   0
 $EndComp
+Wire Wire Line
+	5350 3050 5100 3050
+Wire Wire Line
+	5100 3700 8850 3700
+Wire Wire Line
+	8850 3700 8850 3250
+Wire Wire Line
+	8850 3250 8600 3250
+Wire Wire Line
+	5100 3050 5100 3700
 $EndSCHEMATC
