File: kicad/leds.sch (KiCad schematic (older format))
At the start: 11 parts, among them J14 Ambient_Led_6, J15 Ambient_Led_5, J20 LED_I2C

Commit message: Libraries cleanup
Parts:
- LED1: footprint SamacSys:KRTBLSLPS132VUVXEQBTBVD8TWTZL1B -> KRTBLSLPS132VUVXEQBTBVD8TWTZL1B; symbol SamaSys:KRTBLSLPS1.32-VUVX-EQ+BTBV-D8+TWTZ-L1-B -> SamacSys_Parts:KRTBLSLPS1.32-VUVX-EQ+BTBV-D8+TWTZ-L1-B
- LED2, LED3, LED4: footprint SamacSys:KRTBLSLPS132VUVXEQBTBVD8TWTZL1B -> SamacSys_Parts:KRTBLSLPS132VUVXEQBTBVD8TWTZL1B; symbol SamaSys:KRTBLSLPS1.32-VUVX-EQ+BTBV-D8+TWTZ-L1-B -> SamacSys_Parts:KRTBLSLPS1.32-VUVX-EQ+BTBV-D8+TWTZ-L1-B
- LEDDRV1: footprint SamacSys:QFN40P400X400X100-33N-D -> SamacSys_Parts:QFN40P400X400X100-33N-D; symbol SamaSys:LP5024RSMR -> SamacSys_Parts:LP5024RSMR
Changed lines of the file:
@@
 $Descr A4 11693 8268
 encoding utf-8
-Sheet 5 6
+Sheet 5 7
 Title ""
 Date ""
@@
 Indicator Lights
 $Comp
-L SamaSys:KRTBLSLPS1.32-VUVX-EQ+BTBV-D8+TWTZ-L1-B LED?
+L SamacSys_Parts:KRTBLSLPS1.32-VUVX-EQ+BTBV-D8+TWTZ-L1-B LED?
 U 1 1 601E68E7
 P 2600 1850
@@
 F 0 "LED1" H 3050 1750 50  0000 C CNN
 F 1 "KRTBLSLPS1.32-VUVX-EQ+BTBV-D8+TWTZ-L1-B" H 3050 2024 50  0001 C CNN
-F 2 "SamacSys:KRTBLSLPS132VUVXEQBTBVD8TWTZL1B" H 3350 1950 50  0001 L CNN
+F 2 "KRTBLSLPS132VUVXEQBTBVD8TWTZL1B" H 3350 1950 50  0001 L CNN
 F 3 "https://dammedia.osram.info/media/resource/hires/osram-dam-6176296/KRTB%20LSLPS1.32_EN.pdf" H 3350 1850 50  0001 L CNN
 F 4 "LED RGB 6LED 6PLCC SMD" H 3350 1750 50  0001 L CNN "Description"
@@
 $EndComp
 $Comp
-L SamaSys:KRTBLSLPS1.32-VUVX-EQ+BTBV-D8+TWTZ-L1-B LED?
+L SamacSys_Parts:KRTBLSLPS1.32-VUVX-EQ+BTBV-D8+TWTZ-L1-B LED?
 U 1 1 601E690B
 P 2600 2500
@@
 F 0 "LED2" H 3050 2400 50  0000 C CNN
 F 1 "KRTBLSLPS1.32-VUVX-EQ+BTBV-D8+TWTZ-L1-B" H 3050 2674 50  0001 C CNN
-F 2 "SamacSys:KRTBLSLPS132VUVXEQBTBVD8TWTZL1B" H 3350 2600 50  0001 L CNN
+F 2 "SamacSys_Parts:KRTBLSLPS132VUVXEQBTBVD8TWTZL1B" H 3350 2600 50  0001 L CNN
 F 3 "https://dammedia.osram.info/media/resource/hires/osram-dam-6176296/KRTB%20LSLPS1.32_EN.pdf" H 3350 2500 50  0001 L CNN
 F 4 "LED RGB 6LED 6PLCC SMD" H 3350 2400 50  0001 L CNN "Description"
@@
 $EndComp
 $Comp
-L SamaSys:KRTBLSLPS1.32-VUVX-EQ+BTBV-D8+TWTZ-L1-B LED?
+L SamacSys_Parts:KRTBLSLPS1.32-VUVX-EQ+BTBV-D8+TWTZ-L1-B LED?
 U 1 1 6053070F
 P 2600 3150
@@
 F 0 "LED3" H 3050 3050 50  0000 C CNN
 F 1 "KRTBLSLPS1.32-VUVX-EQ+BTBV-D8+TWTZ-L1-B" H 3050 3324 50  0001 C CNN
-F 2 "SamacSys:KRTBLSLPS132VUVXEQBTBVD8TWTZL1B" H 3350 3250 50  0001 L CNN
+F 2 "SamacSys_Parts:KRTBLSLPS132VUVXEQBTBVD8TWTZL1B" H 3350 3250 50  0001 L CNN
 F 3 "https://dammedia.osram.info/media/resource/hires/osram-dam-6176296/KRTB%20LSLPS1.32_EN.pdf" H 3350 3150 50  0001 L CNN
 F 4 "LED RGB 6LED 6PLCC SMD" H 3350 3050 50  0001 L CNN "Description"
@@
 $EndComp
 $Comp
-L SamaSys:KRTBLSLPS1.32-VUVX-EQ+BTBV-D8+TWTZ-L1-B LED?
+L SamacSys_Parts:KRTBLSLPS1.32-VUVX-EQ+BTBV-D8+TWTZ-L1-B LED?
 U 1 1 6053071B
 P 2600 3800
@@
 F 0 "LED4" H 3050 3700 50  0000 C CNN
 F 1 "KRTBLSLPS1.32-VUVX-EQ+BTBV-D8+TWTZ-L1-B" H 3050 3974 50  0001 C CNN
-F 2 "SamacSys:KRTBLSLPS132VUVXEQBTBVD8TWTZL1B" H 3350 3900 50  0001 L CNN
+F 2 "SamacSys_Parts:KRTBLSLPS132VUVXEQBTBVD8TWTZL1B" H 3350 3900 50  0001 L CNN
 F 3 "https://dammedia.osram.info/media/resource/hires/osram-dam-6176296/KRTB%20LSLPS1.32_EN.pdf" H 3350 3800 50  0001 L CNN
 F 4 "LED RGB 6LED 6PLCC SMD" H 3350 3700 50  0001 L CNN "Description"
@@
 	9850 3200 9450 3200
 $Comp
-L SamaSys:LP5024RSMR LEDDRV?
+L SamacSys_Parts:LP5024RSMR LEDDRV?
 U 1 1 5F3BCCA1
 P 8750 2800
@@
 F 0 "LEDDRV1" V 9400 2450 50  0000 C CNN
 F 1 "LP5024RSMR" V 9550 2450 50  0000 C CNN
-F 2 "SamacSys:QFN40P400X400X100-33N-D" H 10000 3300 50  0001 L CNN
+F 2 "SamacSys_Parts:QFN40P400X400X100-33N-D" H 10000 3300 50  0001 L CNN
 F 3 "http://www.ti.com/lit/gpn/lp5024" H 10000 3200 50  0001 L CNN
 F 4 "24-Channel I2C Constant-Current RGB LED Driver " H 10000 3100 50  0001 L CNN "Description"

Commit message: Comitting yesterday's leftovers
Parts:
- renumbered C1 to C11, C2 to C12, J14 to J10, J15 to J11, J20 to J12, R1 to R16
Connections:
- net VDD renamed +3V3

Commit message: Relabeled and completed ERC
Parts:
- LED1: footprint KRTBLSLPS132VUVXEQBTBVD8TWTZL1B -> SamacSys_Parts:KRTBLSLPS132VUVXEQBTBVD8TWTZL1B
Changed lines of the file:
@@
 F 0 "LED1" H 3050 1750 50  0000 C CNN
 F 1 "KRTBLSLPS1.32-VUVX-EQ+BTBV-D8+TWTZ-L1-B" H 3050 2024 50  0001 C CNN
-F 2 "KRTBLSLPS132VUVXEQBTBVD8TWTZL1B" H 3350 1950 50  0001 L CNN
+F 2 "SamacSys_Parts:KRTBLSLPS132VUVXEQBTBVD8TWTZL1B" H 3350 1950 50  0001 L CNN
 F 3 "https://dammedia.osram.info/media/resource/hires/osram-dam-6176296/KRTB%20LSLPS1.32_EN.pdf" H 3350 1850 50  0001 L CNN
 F 4 "LED RGB 6LED 6PLCC SMD" H 3350 1750 50  0001 L CNN "Description"
