File: kicad/plant_station.kicad_pcb (KiCad board)
At the start: 2 copper layers, 174.4 x 59.3 mm, 147 parts, among them IC1 VEML7700-TT, IC3 TLC555CDR, IC4 ADC081C021CIMK_NOPB, J1 Conn_02x08_Odd_Even, J10 I2C HOST, J11 SOIL_I2C, J12 WEATHER_I2C, J13 MB_I2C, J14 Ambient_Led_6, J15 Ambient_Led_5, J16 Conn_01x06, J17 GPIO, J18 ALWAYS_ON, J19 Ammeter_Jumper, J2 MB_I2C, J20 LED_I2C, J4 MB_I2C, J5 MB_I2C, J6 MB_I2C, J7 Conn_01x08, J8 UART, J9 I2C SCREEN, P1 USB_C_Plug_USB2.0, Q1 DTC113Z, Q3 DTC113Z, Q4 DMG2301L, Q5 BC817DS,115, U1 HDC2010YPAT, U4 ESP-WROOM-02, U5 TPL5110, U6 CP2102N-A01-GQFN28

Commit message: Mapped footprints, PCB in progress
Parts:
- removed D11: 150060VS75000, LED_SMD:LED_0603_1608Metric
- removed D12, D13: LS4148, Parts:MELF_SOD_80_3_BZT55B13GS08
- removed J15: Ambient_Led_5, Parts:Molex_Conn_SMD_01x04_505567_0471
- removed J16: Conn_01x06, Connector_PinHeader_2.54mm:PinHeader_1x06_P2.54mm_Vertical
- removed J17: GPIO, Connector_PinHeader_2.54mm:PinHeader_1x16_P2.54mm_Vertical
- removed J18: ALWAYS_ON, Connector_PinHeader_2.54mm:PinHeader_1x02_P2.54mm_Vertical
- removed J19: Ammeter_Jumper, Connector_PinHeader_2.54mm:PinHeader_1x02_P2.54mm_Vertical
- removed J20: LED_I2C, Parts:Molex_Conn_SMD_01x06_505567_0671
- removed J8: UART, Connector_PinHeader_2.54mm:PinHeader_1x06_P2.54mm_Vertical
- removed P1: USB_C_Plug_USB2.0, Connector_USB:USB_C_Receptacle_Amphenol_12401610E4-2A
- removed Q4: DMG2301L, Package_TO_SOT_SMD:SOT-23
- removed Q5: BC817DS,115, Parts:SOT95P275X110-6N
- removed REF** (x48): Drill Hole, Parts:Drill Hole
- removed REF** (x9): MountingHole_2.2mm_M2_ISO7380, MountingHole:MountingHole_2.2mm_M2_ISO7380
- added BT1: Battery_NTC, Connector_JST:JST_EH_B3B-EH-A_1x03_P2.50mm_Vertical, F.Cu at (245.4, 96.5)
- added C17: 4.7uF, Capacitor_SMD:C_1206_3216Metric, F.Cu at (262.9, 95.5)
- added C18: 1uF, Capacitor_SMD:C_1206_3216Metric, F.Cu at (249.3, 104.7)
- added C19: 0.47uF, Capacitor_SMD:C_1206_3216Metric, F.Cu at (260.6, 102.1)
- added C20: 0.1uF, Capacitor_SMD:C_1206_3216Metric, F.Cu at (255.0, 102.1)
- added C21: 1uF, Capacitor_SMD:C_1206_3216Metric, F.Cu at (244.7, 108.6)
- added D7: 150060VS75000, LED_SMD:LED_0603_1608Metric, F.Cu at (277.5, 128.8)
- added IC2: ADC081C021CIMK_NOPB, SamacSys_Parts:SOT95P280X110-6N, F.Cu at (179.8, 58.4)
- added J3: MB_I2C, Parts:Molex_Conn_SMD_01x06_505567_0671, F.Cu at (254.8, 165.3)
- added Q2: DTC113Z, Parts:DTC113ZEBTL, B.Cu at (221.0, 83.2)
- added R22: 10K, Resistor_SMD:R_0805_2012Metric, F.Cu at (268.9, 130.4)
- added R23: 2K, Resistor_SMD:R_0805_2012Metric, F.Cu at (275.6, 126.1)
- added R24: 2K, Resistor_SMD:R_0805_2012Metric, F.Cu at (267.6, 133.7)
- added R25: 2K, Resistor_SMD:R_0805_2012Metric, F.Cu at (262.6, 136.7)
- added R26: 10K, Resistor_SMD:R_0805_2012Metric, F.Cu at (275.6, 123.1)
- added R27: 37.5K, Resistor_SMD:R_0805_2012Metric, F.Cu at (255.4, 105.3)
- added R28: 1.5K, Resistor_SMD:R_0805_2012Metric, F.Cu at (262.3, 98.7)
- added R29: 1.1K, Resistor_SMD:R_0805_2012Metric, F.Cu at (255.4, 108.2)
- added R30: 1.5K, Resistor_SMD:R_0805_2012Metric, F.Cu at (265.7, 101.6)
- added R31: 1.19K, Resistor_SMD:R_0805_2012Metric, F.Cu at (259.8, 105.3)
- added R32: 10k, Resistor_SMD:R_0805_2012Metric, F.Cu at (259.8, 108.2)
- added R33: 1.8M, Resistor_SMD:R_0805_2012Metric, F.Cu at (264.2, 105.3)
- added SW1: PTS810_SJK_250_SMTR_LFS, Parts:PTS810SJK250SMTRLFS, F.Cu at (287.5, 96.8)
- added SW2: PTS810_SJK_250_SMTR_LFS, Parts:PTS810SJK250SMTRLFS, F.Cu at (287.5, 103.1)
- added U2: SSM6L40TU, Parts:SSM6L40TU, F.Cu at (293.3, 101.2)
- added U3: TPL5110, Package_TO_SOT_SMD:SOT-23-6, F.Cu at (284.7, 111.1)
- added U7: BQ27421YZFR-G1A, Parts:BQ27421YZFR-G1A, F.Cu at (267.5, 108.2)
- added U8: SN74LV00ARGYR, Parts:SN74LV00ARGYR, F.Cu at (256.9, 97.5)
- C1: value 1μF -> 220uF; footprint Capacitor_SMD:C_1206_3216Metric -> Capacitor_Tantalum_SMD:CP_EIA-3216-18_Kemet-A; moved to F.Cu
- C10: value 220uF -> 0.1μF; footprint Capacitor_Tantalum_SMD:CP_EIA-3216-18_Kemet-A -> Capacitor_SMD:C_1206_3216Metric
- C11: value 0.1μF -> 1μF
- C12, C7: value 4.7uF -> 1μF
- C13: value 4.7uF -> 0.1μF
- C14, C6, C9: value 0.1μF -> 4.7uF
- C15: value 0.1μF -> 2.2uF
- C2: value 1μF -> 0.1μF; moved to F.Cu
- C4: value 1μF -> 0.1uF
- C5: value 10nF -> 0.1μF
- C8: value 0.1uF -> 10nF
- D10, D2: value LS4148 -> LED; footprint Parts:MELF_SOD_80_3_BZT55B13GS08 -> LED_SMD:LED_0603_1608Metric
- D3: value 150060AS75000 -> LED
- D4: value 150060BS75020 -> LS4148; footprint LED_SMD:LED_0603_1608Metric -> Parts:MELF_SOD_80_3_BZT55B13GS08
- D5: value SP0503BAHT -> 150060AS75000; footprint Package_TO_SOT_SMD:SOT-143 -> LED_SMD:LED_0603_1608Metric
- D6: value LS4148 -> 150060BS75020; footprint Parts:MELF_SOD_80_3_BZT55B13GS08 -> LED_SMD:LED_0603_1608Metric; moved to F.Cu
- D8: value LS4148 -> SP0503BAHT; footprint Parts:MELF_SOD_80_3_BZT55B13GS08 -> Package_TO_SOT_SMD:SOT-143; moved to F.Cu
- D9: value LS4148 -> LED; footprint Parts:MELF_SOD_80_3_BZT55B13GS08 -> LED_SMD:LED_0603_1608Metric; moved to F.Cu
- IC1: value VEML7700-TT -> TLC555CDR; footprint SamacSys:VEML7700 -> SamacSys_Parts:SOIC127P600X175-8N
- IC3: value TLC555CDR -> VEML7700-TT; footprint SamacSys:SOIC127P600X175-8N -> SamacSys_Parts:VEML7700
- IC4: value ADC081C021CIMK_NOPB -> BQ24079RGTR; footprint SamacSys:SOT95P280X110-6N -> SamacSys_Parts:QFN50P300X300X100-17N-D
- J1: value Conn_02x08_Odd_Even -> MB_I2C; footprint Connector_PinHeader_2.54mm:PinHeader_2x08_P2.54mm_Vertical -> Parts:Molex_Conn_SMD_01x06_505567_0671
- J10: value I2C HOST -> Ambient_Led_6; footprint Connector_PinSocket_2.54mm:PinSocket_1x04_P2.54mm_Vertical -> Parts:Molex_Conn_SMD_01x04_505567_0471; moved to B.Cu
- J11: value SOIL_I2C -> Ambient_Led_5; footprint Parts:Molex_Conn_SMD_01x06_505567_0671 -> Parts:Molex_Conn_SMD_01x04_505567_0471
- J12: value WEATHER_I2C -> LED_I2C
- J13: value MB_I2C -> USB_C_Receptacle_USB2.0; footprint Parts:Molex_Conn_SMD_01x06_505567_0671 -> Parts:CUI_UJ31-CH-3-SMT-TR; moved to F.Cu
- J14: value Ambient_Led_6 -> Ammeter_Jumper; footprint Parts:Molex_Conn_SMD_01x04_505567_0471 -> Connector_PinHeader_2.54mm:PinHeader_1x02_P2.54mm_Vertical; moved to F.Cu
- J2, J4, J5: moved to F.Cu
- J6: value MB_I2C -> I2C; footprint Parts:Molex_Conn_SMD_01x06_505567_0671 -> Connector_PinSocket_2.54mm:PinSocket_1x04_P2.54mm_Vertical; moved to F.Cu
- J7: value Conn_01x08 -> SOIL_I2C; footprint Connector_PinHeader_2.54mm:PinHeader_1x08_P2.54mm_Vertical -> Parts:Molex_Conn_SMD_01x06_505567_0671; moved to B.Cu
- J9: value I2C SCREEN -> WEATHER_I2C; footprint Connector_PinSocket_2.54mm:PinSocket_1x04_P2.54mm_Vertical -> Parts:Molex_Conn_SMD_01x06_505567_0671; moved to B.Cu
- LED1, LED2, LED3, LED4: footprint SamacSys:KRTBLSLPS132VUVXEQBTBVD8TWTZL1B -> SamacSys_Parts:KRTBLSLPS132VUVXEQBTBVD8TWTZL1B
- LEDDRV1: footprint SamacSys:QFN40P400X400X100-33N-D -> SamacSys_Parts:QFN40P400X400X100-33N-D; moved to F.Cu
- Q3: value DTC113Z -> BC817DS,115; footprint Parts:DTC113ZEBTL -> Parts:SOT95P275X110-6N
- R1: value 4K9 -> 10K; moved to F.Cu
- R10: value 10K -> 4.7K
- R12: value 10K -> 16.9K
- R13: value 10K -> 97.6K
- R14: value 1K -> 22
- R15: value 1K -> 1M; footprint Resistor_SMD:R_0805_2012Metric -> Resistor_SMD:R_1206_3216Metric
- R16: value 22K1 -> 4K9
- R17: value 10K -> 47K5
- R18: value 47K5 -> 1K
- R19: value 1K -> 5K1
- R2: value 16.9K -> 2K
- R20: value 10K -> 5K1
- R21: value 10K -> 22K1
- R3: value 4K7 -> 2K
- R4: value 1M -> 10K; footprint Resistor_SMD:R_1206_3216Metric -> Resistor_SMD:R_0805_2012Metric
- R5: value 22 -> 10K
- R6: value 97.6K -> 4K7
- R8: value 1K -> 4K7
- R9: value 4K7 -> 10K
- U1: value HDC2010YPAT -> ESP-WROOM-02; footprint LocalsLib:BGA6C100X50P2X3_146X146X67 -> RF_Module:ESP-WROOM-02
- U4: value ESP-WROOM-02 -> HDC2010YPAT; footprint RF_Module:ESP-WROOM-02 -> Parts:BGA6C100X50P2X3_146X146X67
- U5: value TPL5110 -> CP2102N-A01-GQFN28; footprint Package_TO_SOT_SMD:SOT-23-6 -> Package_DFN_QFN:QFN-28-1EP_5x5mm_P0.5mm_EP3.35x3.35mm
- U6: value CP2102N-A01-GQFN28 -> NCP167BMX330TBG; footprint Package_DFN_QFN:QFN-28-1EP_5x5mm_P0.5mm_EP3.35x3.35mm -> Parts:REG_NCP167BMX330TBG
- moved R2 211.0 mm to (298.9, 103.8), turned to 0 degrees
- moved R6 208.9 mm to (298.9, 106.8), turned to 0 degrees
- moved D2 208.0 mm to (293.6, 113.1), turned to 0 degrees
- moved R13 207.2 mm to (289.3, 110.3), turned to 0 degrees
- moved J6 205.9 mm to (277.2, 151.1), turned to 0 degrees
- moved R7 205.5 mm to (288.9, 116.2), turned to 0 degrees
- moved R9 203.9 mm to (290.1, 106.9), turned to 0 degrees
- moved R3 203.9 mm to (284.4, 117.9), turned to 0 degrees
- moved R12 200.8 mm to (284.4, 114.9), turned to 0 degrees
- moved R10 197.9 mm to (294.5, 104.4), turned to 0 degrees
- moved D8 186.8 mm to (270.9, 123.9), turned to 0 degrees
- moved J5 186.3 mm to (254.8, 158.7), turned to 0 degrees
- moved D6 186.3 mm to (276.3, 131.8), turned to 0 degrees
- moved J2 186.2 mm to (268.2, 158.7), turned to 0 degrees
- moved J4 182.9 mm to (268.2, 152.1), turned to 0 degrees
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Connections:
- C1 pad 1: Net-(C1-Pad1) -> +3V3
- C10 pad 2: GND -> /env_sensor/GND_S
- C12 pad 2: Net-(C11-Pad1) -> +3V3
- C13 pad 1: VDD -> VCC
- C13 pad 2: /env_sensor/GNDA -> GND
- C14 pad 1: VDD -> GND
- C14 pad 2: /env_sensor/GNDA -> VCC
- C16 pad 1: GND -> /charger/BATT
- C16 pad 2: Net-(C15-Pad1) -> GND
- C2 pad 2: VDD -> /esp8266/ESP_RST
- C3 pad 1: /moisture_sensor/GNDA -> GND
- C3 pad 2: /moisture_sensor/VA -> /esp8266/SYS_EN
- C4 pad 1: Net-(C4-Pad1) -> GND
- C4 pad 2: /moisture_sensor/GNDA -> +3V3
- C5 pad 1: Net-(C5-Pad1) -> GNDA
- C5 pad 2: /moisture_sensor/GNDA -> +3.3VA
- C6 pad 1: GND -> +3.3VA
- C6 pad 2: /esp8266/ESP_RST -> GNDA
- C7 pad 1: /moisture_sensor/VA -> Net-(C7-Pad1)
- C7 pad 2: /moisture_sensor/GNDA -> GNDA
- C8 pad 1: GND -> Net-(C8-Pad1)
- C8 pad 2: VDD -> GNDA
- C9 pad 1: GND -> +3V3
- C9 pad 2: /esp8266/ESP_EN -> /env_sensor/GND_S
- Cref1 pad 2: /moisture_sensor/GNDA -> GNDA
- D1 pad 1: Net-(C4-Pad1) -> /ALL_EN
- D1 pad 2: /moisture_sensor/Sensor_Inside -> /esp8266/ALL_EN
- D10 pad 1: Net-(D10-Pad1) -> /charger/CH_PGOOD
- D10 pad 2: /moisture_sensor/ALL_EN -> Net-(D10-Pad2)
- D2 pad 1: Net-(D2-Pad1) -> GND
- D2 pad 2: /esp8266/WAKE_UP -> Net-(D2-Pad2)
- D4 pad 1: /usb_serial/USB_TXT -> Net-(C7-Pad1)
- D4 pad 2: Net-(D4-Pad2) -> /moisture_sensor/Sensor_Inside
- D5 pad 2: Net-(C11-Pad1) -> Net-(D5-Pad2)
- D6 pad 1: Net-(D6-Pad1) -> /usb_serial/USB_TXT
- D6 pad 2: /ALL_EN -> Net-(D6-Pad2)
- D8 pad 1: Net-(D8-Pad1) -> GND
- D8 pad 2: /ALL_EN -> VCC
- D9 pad 2: /ALL_EN -> Net-(D9-Pad2)
- FB1 pad 1: VDD -> +3V3
- FB1 pad 2: /moisture_sensor/VA -> +3.3VA
- FB2 pad 1: Net-(FB2-Pad1) -> GNDA
- FB2 pad 2: GND -> Net-(FB2-Pad2)
- IC1 pad 1: /env_sensor/SCL -> GNDA
- IC1 pad 2: VDD -> Net-(Cref1-Pad1)
- IC1 pad 3: /env_sensor/GNDA -> /moisture_sensor/Sensor_Inside
- IC1 pad 4: /env_sensor/SDA -> +3.3VA
- IC3 pad 1: /moisture_sensor/GNDA -> /env_sensor/SCL
- IC3 pad 2: Net-(Cref1-Pad1) -> +3V3
- IC3 pad 3: /moisture_sensor/Sensor_Inside -> /env_sensor/GND_S
- IC3 pad 4: /moisture_sensor/VA -> /env_sensor/SDA
- IC4 pad 1: /moisture_sensor/VA -> /charger/BATT_T
- IC4 pad 2: /moisture_sensor/GNDA -> /charger/BATT
- IC4 pad 3: Net-(IC4-Pad3) -> /charger/BATT
- IC4 pad 4: /moisture_sensor/HOST_WAKE -> /charger/CH_PGOOD
- IC4 pad 5: /moisture_sensor/SCL -> /charger/CH_EN2
- IC4 pad 6: /moisture_sensor/SDA -> /charger/CH_EN1
- J1 pad 1: /esp8266/WAKE_UP -> GND
- J1 pad 2: /esp8266/GPIO16 -> +3V3
- J1 pad 3: VDD -> /SDA
- J1 pad 4: +3V3 -> /SCL
- J1 pad 5: VDD -> /HOST_WAKE_UP
- J1 pad 6: Net-(J1-Pad12) -> /ALL_EN
- J10 pad 1: GND -> /leds/LED_3_B
- J10 pad 2: VDD -> /leds/LED_3_G
- J10 pad 3: /SCL -> /leds/LED_3_R
- J10 pad 4: /SDA -> +3V3
- J11 pad 1: GND -> /leds/LED_4_B
- J11 pad 2: VDD -> /leds/LED_4_G
- J11 pad 3: /moisture_sensor/SDA -> /leds/LED_4_R
- J11 pad 4: /moisture_sensor/SCL -> +3V3
- J11 pad 5: /moisture_sensor/HOST_WAKE -> Net-(J11-Pad5)
- J11 pad 6: /moisture_sensor/ALL_EN -> Net-(J11-Pad6)
- J12 pad 2: VDD -> +3V3
- J12 pad 3: /env_sensor/SDA -> /leds/SDA
- J12 pad 4: /env_sensor/SCL -> /leds/SCL
- J12 pad 6: /env_sensor/ALL_EN -> /leds/ALL_EN
- J14 pad 1: /leds/LED_3_B -> Net-(C15-Pad1)
- J14 pad 2: /leds/LED_3_G -> +3V3
- J2 pad 2: VDD -> +3V3
- J2 pad 5: /HOST_WAKE -> /HOST_WAKE_UP
- J2 pad 6: Net-(D6-Pad1) -> /ALL_EN
- J4 pad 2: VDD -> +3V3
- J4 pad 5: /HOST_WAKE -> /HOST_WAKE_UP
- J4 pad 6: Net-(D12-Pad1) -> /ALL_EN
- J5 pad 2: VDD -> +3V3
- J5 pad 5: /HOST_WAKE -> /HOST_WAKE_UP
- J5 pad 6: Net-(D8-Pad1) -> /ALL_EN
- J6 pad 2: VDD -> +3V3
- J6 pad 3: /SDA -> /SCL
- J6 pad 4: /SCL -> /SDA
- J7 pad 1: /usb_serial/USB_DTR -> GND
- J7 pad 2: /usb_serial/USB_DSR -> +3V3
- J7 pad 3: /usb_serial/USB_RTS -> /moisture_sensor/SDA
- J7 pad 4: /usb_serial/USB_CTS -> /moisture_sensor/SCL
- J7 pad 5: /usb_serial/USB_GPIO.4 -> /moisture_sensor/HOST_WAKE
- J7 pad 6: /usb_serial/USB_GPIO.5 -> /moisture_sensor/ALL_EN
- J9 pad 2: VDD -> +3V3
- J9 pad 3: /SCL -> /env_sensor/SDA
- J9 pad 4: /SDA -> /env_sensor/SCL
- LED1 pad A1: VDD -> +3V3
- LED1 pad A2: VDD -> +3V3
- LED1 pad A3: VDD -> +3V3
- LED2 pad A1: VDD -> +3V3
- LED2 pad A2: VDD -> +3V3
- LED2 pad A3: VDD -> +3V3
- LED3 pad A1: VDD -> +3V3
- LED3 pad A2: VDD -> +3V3
- LED3 pad A3: VDD -> +3V3
- LED4 pad A1: VDD -> +3V3
- LED4 pad A2: VDD -> +3V3
- LED4 pad A3: VDD -> +3V3
- LEDDRV1 pad 27: VDD -> +3V3
- LEDDRV1 pad 32: Net-(C1-Pad1) -> Net-(C11-Pad1)
- Q1 pad 1: Net-(D10-Pad1) -> /moisture_sensor/ALL_EN
- Q1 pad 2: Net-(FB2-Pad1) -> GND
- Q1 pad 3: /moisture_sensor/GNDA -> Net-(FB2-Pad2)
- Q3 pad 1: /env_sensor/ALL_EN -> /usb_serial/USB_RTS
- Q3 pad 2: GND -> Net-(Q3-Pad2)
- Q3 pad 3: /env_sensor/GNDA -> /esp8266/BOOT_MODE
- R1 pad 1: GND -> +3V3
- R1 pad 2: Net-(LEDDRV1-Pad31) -> /esp8266/ESP_RST
- R10 pad 1: +3V3 -> Net-(R10-Pad1)
- R10 pad 2: /esp8266/ESP_RST -> GND
- R11 pad 1: Net-(R11-Pad1) -> +3V3
- R11 pad 2: GND -> Net-(R11-Pad2)
- R12 pad 1: GND -> /esp8266/TPL_MDRV
- R12 pad 2: /esp8266/GPIO15 -> GND
- R13 pad 1: +3V3 -> /esp8266/TPL_MDRV
- R13 pad 2: /esp8266/GPIO0 -> GND
- R14 pad 1: Net-(C11-Pad1) -> Net-(IC2-Pad3)
- R14 pad 2: Net-(D4-Pad2) -> Net-(C7-Pad1)
- R15 pad 1: Net-(C11-Pad1) -> Net-(C7-Pad1)
- R15 pad 2: Net-(D11-Pad2) -> GNDA
- R16 pad 1: Net-(R16-Pad1) -> GND
- R16 pad 2: Net-(C11-Pad1) -> Net-(LEDDRV1-Pad31)
- R17 pad 1: /esp8266/ESP_EN -> Net-(R17-Pad1)
- R17 pad 2: Net-(J1-Pad12) -> GND
- R18 pad 1: Net-(R16-Pad1) -> VCC
- R18 pad 2: GND -> Net-(R18-Pad2)
- R19 pad 1: Net-(C15-Pad1) -> GND
- R19 pad 2: Net-(R19-Pad2) -> Net-(J13-PadA5)
- R2 pad 1: Net-(D2-Pad1) -> Net-(D2-Pad2)
- R2 pad 2: GND -> /esp8266/SYS_EN
- R20 pad 1: Net-(Q5-Pad5) -> GND
- R20 pad 2: /usb_serial/USB_RTS -> Net-(J13-PadB5)
- R21 pad 1: /usb_serial/USB_DTR -> Net-(R17-Pad1)
- R21 pad 2: Net-(Q5-Pad2) -> VCC
- R3 pad 1: VDD -> Net-(D3-Pad2)
- R3 pad 2: /SDA -> +3V3
- R4 pad 1: Net-(C4-Pad1) -> +3V3
- R4 pad 2: /moisture_sensor/GNDA -> /esp8266/BOOT_MODE
- R5 pad 1: Net-(IC4-Pad3) -> GND
- R5 pad 2: Net-(C4-Pad1) -> /esp8266/GPIO15
- R6 pad 1: Net-(D2-Pad1) -> +3V3
- R6 pad 2: GND -> /SDA
- R7 pad 2: /esp8266/WAKE_UP -> /HOST_WAKE_UP
- R8 pad 1: Net-(C11-Pad1) -> +3V3
- R8 pad 2: Net-(D3-Pad2) -> /SCL
- R9 pad 1: VDD -> Net-(R9-Pad1)
- R9 pad 2: /SCL -> +3V3
- Ra1 pad 1: /moisture_sensor/VA -> +3.3VA
- Ra1 pad 2: Net-(IC3-Pad7) -> Net-(IC1-Pad7)
- Rb1 pad 1: Net-(IC3-Pad7) -> Net-(IC1-Pad7)
- U5 pad 1: VDD -> Net-(U5-Pad1)
- U5 pad 2: GND -> Net-(U5-Pad2)
- U5 pad 3: Net-(D2-Pad1) -> GND
- U5 pad 4: Net-(J1-Pad13) -> /usb_serial/D+
- U5 pad 5: Net-(J1-Pad11) -> /usb_serial/D-
- U5 pad 6: VDD -> VCC
- U6 pad 1: Net-(U6-Pad1) -> Net-(C15-Pad1)
- U6 pad 2: Net-(U6-Pad2) -> GND
- U6 pad 3: GND -> Net-(C17-Pad1)
- U6 pad 4: /usb_serial/D+ -> Net-(C17-Pad1)
- U6 pad 5: /usb_serial/D- -> GND
Routing:
- net GND: track 312.1 -> 36.5 mm, vias 23 -> 2
- net VDD: track 266.7 -> 0.00 mm, vias 13 -> 0
- net /SCL: track 172.9 -> 0.00 mm, vias 2 -> 0
- net /SDA: track 161.1 -> 0.00 mm, vias 2 -> 0
- net /ALL_EN: track 147.2 -> 0.00 mm, vias 1 -> 0
- net /HOST_WAKE: track 130.7 -> 0.00 mm
- net /esp8266/WAKE_UP: track 81.6 -> 0.00 mm, vias 1 -> 0
- net /esp8266/ESP_EN: track 79.5 -> 0.00 mm, vias 2 -> 0
- net /esp8266/GPIO5: track 61.5 -> 0.00 mm, vias 2 -> 0
- net /esp8266/ESP_RST: track 57.7 -> 0.00 mm, vias 1 -> 0
- net Net-(C11-Pad1): track 54.6 -> 2.44 mm
- net /esp8266/USB_RXD: track 47.3 -> 0.00 mm, vias 1 -> 0
- net /esp8266/GPIO16: track 47.3 -> 0.00 mm
- net /esp8266/USB_TXD: track 45.4 -> 0.00 mm, vias 1 -> 0
- net GNDA: track 0.00 -> 39.0 mm, vias 0 -> 2
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- added copper zone on F.Cu, net +3V3
- added copper zone on B.Cu, net /env_sensor/GND_S
- added copper zone on B.Cu, net GNDA
- added copper zone on F.Cu, net GNDA
- removed copper zone on B.Cu, net (none)
- removed copper zone on B.Cu, net /moisture_sensor/GNDA
- removed copper zone on F.Cu, net /moisture_sensor/GNDA
- removed copper zone on F.Cu, net /moisture_sensor/VA
- removed copper zone on B.Cu, net GND
- removed copper zone on F.Cu, net GND
- removed copper zone on B.Cu, net VDD
- removed copper zone on F.Cu, net VDD
Other:
- board size 174.4 x 59.3 mm -> 80.8 x 113 mm
- board text removed: "The hole on the LEDs screen is missing. And mirror the holes!"
